File: hardware/kicad/SHT41-Sensor-Breakout.kicad_sch (KiCad schematic)
At the start: 56 parts, among them J1 Conn_01x02_Socket, J2 524372771, J3 Conn_02x05_Odd_Even, J4 MicroSD_SPI_Module, SW1 SW_Push_Dual_x2, U1 STM32L431CBT6, U2 SHT41

Commit message: docs: update schematic title block
Other:
- title: STM32 SHT41 Environmental Logger -> STM32 Environmental Logger
Changed lines of the file:
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@@
 	(paper "B")
 	(title_block
-		(title "STM32 SHT41 Environmental Logger")
+		(title "STM32 Environmental Logger")
 		(date "2026-06-23")
 		(rev "A")
